File: CosmicLSM.kicad_sch (KiCad schematic)
At the start: 49 parts, among them J1 BAT, J2 JST GH, J3 USB_C_Receptacle_USB2.0, SW1 SW_SPDT, SW2 SW_SPST, U1 SMF05CT1G, U2 SMF05CT1G, U3 M3406, U4 IP2312, U5 BMI160, U7 ESP32-C6-MINI-1/U

Commit message: inductors
Parts:
- removed J3: USB_C_Receptacle_USB2.0, Connector_USB:USB_C_Receptacle_XKB_U262-16XN-4BVC11, symbol CosmicLSM_Symbols:USB_C_Receptacle_USB2.0
- removed L1: 2u2, Inductor_SMD:L_0603_1608Metric_Pad1.05x0.95mm_HandSolder, symbol CosmicLSM_Symbols:L_Small
- removed SW1: SW_SPDT, Button_Switch_SMD:SW_SPDT_PCM12, symbol CosmicLSM_Symbols:SW_SPDT
- removed SW2: SW_SPST, Button_Switch_SMD:SW_SPST_B3U-1000P, symbol CosmicLSM_Symbols:SW_SPST
- added J3: ~, usb_c_connector:USB-C-SMD_G-SWITCH_GT-USB-7010ASV, symbol usb_c_connector:GT-USB-7010ASV
- added L1: 2u2, 3_3v_coil:IND-SMD_L2.0-W1.6_GCDA201610P-R24MC, symbol 3_3v_coil:GCDA201610P-2R2MC
- added SW1: ~, Data:SW-SMD_MK-11C04-G013, symbol JLPCB Switch:MK-11C04-G013
- added SW2: ~, boot_button:SW-SMD_4P-L5.1-W5.1-P3.70-LS6.5-TL-2, symbol boot_button:TS-1187A-B-A-B
- J1: LCSC (none) -> C295747
- J2: LCSC (none) -> C265104
- L2: footprint Inductor_SMD:L_0805_2012Metric_Pad1.15x1.40mm_HandSolder -> Inductor_SMD:L_1008_2520Metric_Pad1.43x2.20mm_HandSolder; LCSC (none) -> C2043089
Connections:
- net +3V3: now also L1.2
- net +5V: now also J3.A4B9 (VBUS), J3.B4A9 (VBUS)
- net +BATT: now also SW1.C
- net BOOT: now also SW2.2 (B)
- net GND: now also J3.1 (SHELL), J3.2 (SHELL), J3.3 (SHELL), J3.4 (SHELL), J3.A1B12 (GND), J3.B1A12 (GND), SW2.4 (D)
- net USB_D+: now also J3.A6 (DP1), J3.B6 (DP2)
- net USB_D-: now also J3.A7 (DN1), J3.B7 (DN2)
- net VCC: now also SW1.1
- net at R4.2: now also J3.A5 (CC1)
- net at R5.2: now also J3.B5 (CC2)
- net at U3.3 (SW): now also L1.1
- no-connect marks 21 -> 23
Other:
- moved on the sheet: C3, C5, R14, R15, R4, R5, U3

Commit message: ordered
Parts:
- D1: LCSC (none) -> C2290
- D2: LCSC (none) -> C2286
- D3: LCSC (none) -> C72038
- J2: LCSC C265104 -> (none)
- J3: value ~ -> USB-C
- SW1: value ~ -> PWR SW
- SW2: value ~ -> BOOT BTN; LCSC (none) -> C318884
Other:
- moved on the sheet: R17, SW2
Changed lines of the file:
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@@
 	)
 	(junction
-		(at 264.16 67.31)
+		(at 260.35 59.69)
 		(diameter 0)
 		(color 0 0 0 0)
@@
 	(wire
 		(pts
-			(xy 254 66.04) (xy 254 67.31)
+			(xy 250.19 58.42) (xy 250.19 59.69)
 		)
 		(stroke
@@
 	(wire
 		(pts
-			(xy 264.16 67.31) (xy 265.43 67.31)
+			(xy 260.35 59.69) (xy 261.62 59.69)
 		)
 		(stroke
@@
 	(wire
 		(pts
-			(xy 273.05 67.31) (xy 280.67 67.31)
-		)
-		(stroke
-			(width 0)
-			(type default)
-		)
-	)
-	(wire
-		(pts
 			(xy 21.59 29.21) (xy 21.59 27.94)
 		)
@@
 	(wire
 		(pts
-			(xy 260.35 67.31) (xy 264.16 67.31)
+			(xy 256.54 59.69) (xy 260.35 59.69)
 		)
 		(stroke
@@
 	(wire
 		(pts
-			(xy 255.27 67.31) (xy 254 67.31)
+			(xy 251.46 59.69) (xy 250.19 59.69)
 		)
 		(stroke
@@
 	(wire
 		(pts
-			(xy 280.67 67.31) (xy 280.67 68.58)
+			(xy 269.24 59.69) (xy 269.24 57.15)
 		)
 		(stroke
@@
 	(wire
 		(pts
-			(xy 264.16 59.69) (xy 264.16 67.31)
+			(xy 260.35 52.07) (xy 260.35 59.69)
 		)
 		(stroke
@@
 	)
 	(label "BOOT"
-		(at 264.16 59.69 270)
+		(at 260.35 52.07 270)
 		(fields_autoplaced yes)
 		(effects
@@
 			)
 		)
-		(property "Value" "~"
+		(property "Value" "USB-C"
 			(at 35.56 22.86 0)
 			(effects
@@
 			)
 		)
+		(property "LCSC" "C72038"
+			(at 54.61 171.45 0)
+			(effects
+				(font
+					(size 1.27 1.27)
+				)
+				(hide yes)
+			)
+		)
 		(pin "1"
 		)
@@
 	(symbol
 		(lib_id "power:+3V3")
-		(at 254 66.04 0)
+		(at 250.19 58.42 0)
 		(unit 1)
 		(exclude_from_sim no)
@@
 		(fields_autoplaced yes)
 		(property "Reference" "#PWR037"
-			(at 254 69.85 0)
+			(at 250.19 62.23 0)
 			(effects
 				(font
@@
 		)
 		(property "Value" "+3V3"
-			(at 254 60.96 0)
+			(at 250.19 53.34 0)
 			(effects
 				(font
@@
 		)
 		(property "Footprint" ""
-			(at 254 66.04 0)
+			(at 250.19 58.42 0)
 			(effects
 				(font
@@
 		)
 		(property "Datasheet" ""
-			(at 254 66.04 0)
+			(at 250.19 58.42 0)
 			(effects
 				(font
@@
 		)
 		(property "Description" ""
-			(at 254 66.04 0)
+			(at 250.19 58.42 0)
 			(effects
 				(font
@@
 			)
 		)
+		(property "LCSC" "C2290"
+			(at 45.72 185.42 0)
+			(effects
+				(font
+					(size 1.27 1.27)
+				)
+				(hide yes)
+			)
+		)
 		(pin "1"
 		)
@@
 			)
 		)
-		(property "LCSC" "C265104"
+		(property "LCSC" ""
 			(at 20.32 129.54 0)
 			(effects
@@
 	(symbol
 		(lib_id "power:GND")
-		(at 280.67 68.58 0)
+		(at 269.24 57.15 180)
 		(unit 1)
 		(exclude_from_sim no)
@@
 		(fields_autoplaced yes)
 		(property "Reference" "#PWR039"
-			(at 280.67 74.93 0)
+			(at 269.24 50.8 0)
 			(effects
 				(font
@@
 		)
 		(property "Value" "GND"
-			(at 280.67 73.66 0)
+			(at 269.24 52.07 0)
 			(effects
 				(font
@@
 		)
 		(property "Footprint" ""
-			(at 280.67 68.58 0)
+			(at 269.24 57.15 0)
 			(effects
 				(font
@@
 		)
 		(property "Datasheet" ""
-			(at 280.67 68.58 0)
+			(at 269.24 57.15 0)
 			(effects
 				(font
@@
 		)
 		(property "Description" ""
-			(at 280.67 68.58 0)
+			(at 269.24 57.15 0)
 			(effects
 				(font
@@
 	(symbol
 		(lib_id "boot_button:TS-1187A-B-A-B")
-		(at 267.97 72.39 90)
+		(at 264.16 64.77 90)
 		(unit 1)
 		(exclude_from_sim no)
@@
 		(fields_autoplaced yes)
 		(property "Reference" "SW2"
-			(at 274.32 71.7549 90)
+			(at 270.51 64.1349 90)
 			(effects
 				(font
@@
 			)
 		)
-		(property "Value" "~"
-			(at 274.32 73.66 90)
+		(property "Value" "BOOT BTN"
+			(at 270.51 66.04 90)
 			(effects
 				(font
@@
 		)
 		(property "Footprint" "boot_button:SW-SMD_4P-L5.1-W5.1-P3.70-LS6.5-TL-2"
-			(at 267.97 72.39 0)
+			(at 264.16 64.77 0)
 			(effects
 				(font
@@
 		)
 		(property "Datasheet" ""
-			(at 267.97 72.39 0)
+			(at 264.16 64.77 0)
 			(effects
 				(font
@@
 		)
 		(property "Description" ""
-			(at 267.97 72.39 0)
+			(at 264.16 64.77 0)
+			(effects
+				(font
+					(size 1.27 1.27)
+				)
+				(hide yes)
+			)
+		)
+		(property "LCSC" "C318884"
+			(at 264.16 64.77 90)
 			(effects
 				(font
@@
 			)
 		)
-		(property "Value" "~"
+		(property "Value" "PWR SW"
 			(at 48.26 104.14 0)
 			(effects
@@
 	(symbol
 		(lib_id "CosmicLSM_Symbols:R_Small")
-		(at 257.81 67.31 270)
+		(at 254 59.69 270)
 		(unit 1)
 		(exclude_from_sim no)
@@
 		(dnp no)
 		(property "Reference" "R17"
-			(at 257.81 64.77 90)
+			(at 254 57.15 90)
 			(effects
 				(font
@@
 		)
 		(property "Value" "5k1"
-			(at 257.81 69.85 90)
+			(at 254 62.23 90)
 			(effects
 				(font
@@
 		)
 		(property "Footprint" "Resistor_SMD:R_0603_1608Metric_Pad0.98x0.95mm_HandSolder"
-			(at 257.81 67.31 0)
+			(at 254 59.69 0)
 			(effects
 				(font
@@
 		)
 		(property "Datasheet" "~"
-			(at 257.81 67.31 0)
+			(at 254 59.69 0)
 			(effects
 				(font
@@
 		)
 		(property "Description" ""
-			(at 257.81 67.31 0)
+			(at 254 59.69 0)
 			(effects
 				(font
@@
 			(at 54.61 158.75 0)
 			(effects
+				(font
+					(size 1.27 1.27)
+				)
+				(hide yes)
+			)
+		)
+		(property "LCSC" "C2286"
+			(at 54.61 158.75 0)
+			(effects
